File: tool_board/IO.kicad_sch (KiCad schematic)
At the start: 5 parts, among them J4 Conn_01x08_Socket, J5 Fan, J6 Temperature Read 1, J7 Temperature Read 2, J8 Driver

Commit message: message
Parts:
- removed J8: Driver, symbol Connector_Generic:Conn_02x08_Counter_Clockwise
- added J2: 24V Bus, Connector_Phoenix_MC:PhoenixContact_MCV_1,5_2-G-3.5_1x02_P3.50mm_Vertical, symbol Connector:Conn_01x02_Socket
- added J3: DRIVER_POWER_RIAL, Connector_PinSocket_2.54mm:PinSocket_1x08_P2.54mm_Vertical, symbol Connector:Conn_01x08_Socket
- added J8: STP_DIR_EN_BUS, Connector_PinSocket_2.54mm:PinSocket_1x08_P2.54mm_Vertical, symbol Connector:Conn_01x08_Socket
- added J9: MOTOR_OUTPUT, Connector_PinSocket_2.54mm:PinSocket_1x04_P2.54mm_Horizontal, symbol Connector:Conn_01x04_Socket
- J4: footprint (none) -> Connector_RJ:RJ45_OST_PJ012-8P8CX_Vertical
- J5: footprint (none) -> Connector_PinHeader_2.54mm:PinHeader_1x03_P2.54mm_Vertical
- J6, J7: footprint (none) -> Connector_PinHeader_2.54mm:PinHeader_1x02_P2.54mm_Vertical
Connections:
- net +5V: now also J3.7 (Pin_7)
- net A+: now also J3.6 (Pin_6), J9.1 (Pin_1)
- net A-: now also J3.5 (Pin_5), J9.2 (Pin_2)
- net B+: now also J3.4 (Pin_4), J9.3 (Pin_3)
- net B-: now also J3.3 (Pin_3), J9.4 (Pin_4)
- net DIR : now also J8.8 (Pin_8)
- net EN  : now also J8.1 (Pin_1)
- net GND: now also J2.2 (Pin_2), J3.2 (Pin_2), J3.8 (Pin_8)
- net STEP: now also J8.7 (Pin_7)
- net 24v renamed +24V
- net +24V: now also J2.1 (Pin_1), J3.1 (Pin_1)
- no-connect marks 0 -> 5
