File: tool_board/arduinocrystal.kicad_sch (KiCad schematic)
At the start: 4 parts, among them Y1 ABLS-12.000MHZ-B4-T

Commit message: message
Parts:
- C6, C7: footprint (none) -> Capacitor_SMD:C_0805_2012Metric_Pad1.18x1.45mm_HandSolder
- R4: footprint (none) -> Resistor_SMD:R_0612_1632Metric_Pad1.18x3.40mm_HandSolder
- Y1: footprint (none) -> Crystal:Crystal_AT310_D3.0mm_L10.0mm_Horizontal
Changed lines of the file:
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@@
   )
   (text "Crystal Oscillator\n-----------------------------------------\nHowever, as the frequency of this internal oscillator is \nnot well defined or controlled, varying from chip to chip, \nas well as with different supply voltages and temperatures, \nit is recommended to use a stable external frequency source.\n\nProviding an external frequency source can be done in one of \ntwo ways: either by providing a clock source with a CMOS\noutput (3.3V square wave) into the XIN pin, or by using a \n12MHz crystal connected between XIN and XOUT. Using a\ncrystal is the preferred option here, as they are both relatively \ncheap and very accurate.\n\nThe chosen crystal for this design is an ABLS-12.000MHZ-B4-T. This \nis a commonly available 12MHz crystal with a 30ppm tolerance, which \nshould be good enough for most applications. This device also has a \nmaximumESR of 50Ω, and a load capacitance of 18pF, both of which have \na bearing on the choice of accompanying components."
-    (at 135.89 66.04 0)
+    (at 109.22 66.04 0)
     (effects (font (size 1.27 1.27)) (justify left bottom))
   )
@@
       (effects (font (size 1.27 1.27)) (justify right))
     )
-    (property "Footprint" "" (at 58.42 40.64 0)
+    (property "Footprint" "Crystal:Crystal_AT310_D3.0mm_L10.0mm_Horizontal" (at 58.42 40.64 0)
       (effects (font (size 1.27 1.27)) hide)
     )
@@
       (effects (font (size 1.27 1.27)))
     )
-    (property "Footprint" "" (at 41.91 47.9552 0)
+    (property "Footprint" "Capacitor_SMD:C_0805_2012Metric_Pad1.18x1.45mm_HandSolder" (at 41.91 47.9552 0)
       (effects (font (size 1.27 1.27)) hide)
     )
@@
       (effects (font (size 1.27 1.27)))
     )
-    (property "Footprint" "" (at 41.91 36.5252 0)
+    (property "Footprint" "Capacitor_SMD:C_0805_2012Metric_Pad1.18x1.45mm_HandSolder" (at 41.91 36.5252 0)
       (effects (font (size 1.27 1.27)) hide)
     )
@@
       (effects (font (size 1.27 1.27)))
     )
-    (property "Footprint" "" (at 68.834 45.974 90)
+    (property "Footprint" "Resistor_SMD:R_0612_1632Metric_Pad1.18x3.40mm_HandSolder" (at 68.834 45.974 90)
       (effects (font (size 1.27 1.27)) hide)
     )
