File: tool_board/tool_board.kicad_sch (KiCad schematic)
At the start: 5 parts, among them U1 ATmega328P-P

Commit message: message
Parts:
- C3, C4, C5, C6: footprint (none) -> Capacitor_SMD:C_0805_2012Metric_Pad1.18x1.45mm_HandSolder
- U1: footprint Package_DIP:DIP-28_W7.62mm -> Package_QFP:LQFP-32_7x7mm_P0.8mm
Connections:
- net +5V: now also C3.1, C4.1, C5.1, C6.1; no longer C3.2, C4.2, C5.2, C6.2, U1.22 (GND), U1.8 (GND)
- net ETH0: now also U1.25 (PC2); no longer U1.2 (PD0)
- net ETH1: now also U1.26 (PC3); no longer U1.3 (PD1)
- net Reset: now reaches U1.1 (~{RESET}/PC6)
- net EN  : now reaches U1.16 (PB2)
- net STEP: now reaches U1.17 (PB3)
- net DIR : now reaches U1.18 (PB4)
- new net GND: C3.2, C4.2, C5.2, C6.2, U1.22 (GND), U1.8 (GND)
- new net RXD: U1.3 (PD1)
- new net TXD: U1.2 (PD0)
- no-connect marks 0 -> 4
Other:
- moved on the sheet: C3, C4, C5, C6, U1
