File: DigitalWeldReader-Henry/DigitalWeldReader-Henry.kicad_sch (KiCad schematic)
At the start: 38 parts, among them J1 Input Plug, J2 Output Plug, Q1 BSS138, Q2 BSS138, Q3 BSS138, Q4 BSS138, U1 4N25, U2 4N25, U3 4N25, U4 4N25

Commit message: back from break
Parts:
- removed D1, D10, D11: LED, LED_SMD:LED_0603_1608Metric, symbol Device:LED
- removed D12, D3, D6, D9: BAT54SW, Package_TO_SOT_SMD:SOT-323_SC-70, symbol Diode:BAT54SW
- removed R2, R6: R_US, Resistor_SMD:R_0402_1005Metric, symbol Device:R_US
- removed R5: 330, Resistor_SMD:R_0402_1005Metric, symbol Device:R_US
- removed U2, U3: 4N25, Package_DIP:DIP-6_W7.62mm, symbol Isolator:4N25
- added D3, D6, D9: LED, LED_SMD:LED_0603_1608Metric, symbol Device:LED
- added Q5, Q6, Q7, Q8: BSS138, Package_TO_SOT_SMD:SOT-23, symbol Transistor_FET:BSS138
- added R17, R20, R23, R26: 140, Resistor_SMD:R_0402_1005Metric, symbol Device:R_US
- added R18, R21, R24, R27: 220, Resistor_SMD:R_0402_1005Metric, symbol Device:R_US
- added R19, R22, R25: 330, Resistor_SMD:R_0402_1005Metric, symbol Device:R_US
- added U10, U11, U6, U7, U8, U9: 4N25, Package_DIP:DIP-6_W7.62mm, symbol Isolator:4N25
- J1: value Input Plug -> Signal Input Plug; footprint Connector_Phoenix_MC:PhoenixContact_MC_1,5_6-GF-3.81_1x06_P3.81mm_Horizontal_ThreadedFlange_MountHole -> Connector_Phoenix_MC:PhoenixContact_MC_1,5_8-GF-3.81_1x08_P3.81mm_Horizontal_ThreadedFlange; symbol Connector_Generic:Conn_01x06 -> Connector_Generic:Conn_01x08
- J2: footprint Connector_Phoenix_MC:PhoenixContact_MC_1,5_6-GF-3.81_1x06_P3.81mm_Horizontal_ThreadedFlange_MountHole -> Connector_RJ:RJ45_Amphenol_54602-x08_Horizontal; symbol Connector_Generic:Conn_01x06 -> Connector_Generic:Conn_01x08
- R10: value R_US -> 330
- R12, R3: value 2k05 -> 220
- R14: value R_US -> 140
- R15: value 140 -> 220
- R16: value 2k05 -> 330
- R7: value 140 -> 330
- R8: value 2k05 -> 140
- R9: value 330 -> 220
Connections:
- net +24V: now also R11.2, R14.2, R4.2, R8.2, R17.2, R20.2, R23.2, R26.2; no longer J2.6 (Pin_6), U1.5, U4.5
- net +5V: now also U1.5, U4.5, U10.5, U11.5, U6.5, U7.5, U8.5, U9.5; no longer J1.1 (Pin_1), R11.2, R15.2, R4.2, R7.2
- net GND1: now also Q1.2 (S), Q2.2 (S), Q3.2 (S), Q4.2 (S), Q5.2 (S), Q6.2 (S), Q7.2 (S), Q8.2 (S); no longer J1.6 (Pin_6), R10.1, R14.1
- net GND2: now also R15.1, R9.1, R18.1, R21.1, R24.1, R27.1; no longer J2.1 (Pin_1), R16.1, R8.1
- net IN1: now also J1.1 (Pin_1), R1.1; no longer J1.3 (Pin_3)
- net IN2: now also J1.2 (Pin_2), R7.1; no longer J1.4 (Pin_4), R9.1
- net IN3: now also J1.3 (Pin_3), R10.1; no longer J1.5 (Pin_5), R13.1
- net OUT1: now also D2.2 (A), J2.1 (Pin_1), U1.4; no longer D5.2 (A), J2.4 (Pin_4)
- net OUT2: now also J2.2 (Pin_2), U4.4, D3.2 (A); no longer J2.3 (Pin_3)
- net OUT3: now also D4.2 (A), J2.3 (Pin_3), U6.4; no longer J2.2 (Pin_2), U4.4
- net at R16.2: now also Q5.1 (G)
- net at R12.2: now also D4.1 (K); no longer D8.1 (K)
- net OUT7: now reaches D8.2 (A)
- net OUT7: now also J2.7 (Pin_7), U10.4
- net at Q3.1 (G): now also R10.2; no longer R9.2
- net at Q2.1 (G): now also R7.2
- net at D5.1 (K): now also R15.2; no longer R8.2
- net at R11.1: now also U6.1
- net at Q2.3 (D): now also U4.2
- net at Q3.3 (D): now also U6.2
- net at D7.1 (K): now also R21.2; no longer R10.2
- net at U4.1: now also R8.1; no longer R15.1
- net at Q4.3 (D): now also U7.2; no longer U4.2
- net OUT6: now reaches D7.2 (A)
- net OUT6: now also J2.6 (Pin_6), U9.4; no longer Q3.2 (S)
- removed net IN0: J1.2 (Pin_2), R1.1
- removed net OUT0: D2.2 (A), J2.5 (Pin_5), U1.4
- new net: D9.1 (K), R27.2
- new net: Q6.1 (G), R19.2
- new net: Q6.3 (D), U9.2
- new net: Q7.1 (G), R22.2
- new net: R23.1, U10.1
- new net: Q8.1 (G), R25.2
- new net: Q8.3 (D), U11.2
- new net: Q5.3 (D), U8.2
- new net: R17.1, U8.1
- new net: Q7.3 (D), U10.2
- new net: D6.1 (K), R18.2
- new net: R14.1, U7.1
- new net: R26.1, U11.1
- new net: R20.1, U9.1
- new net: D3.1 (K), R9.2
- new net: D8.1 (K), R24.2
- new net IN4: J1.4 (Pin_4), R13.1
- new net IN5: J1.5 (Pin_5), R16.1
- new net IN6: J1.6 (Pin_6), R19.1
- new net IN7: J1.7 (Pin_7), R22.1
- new net IN8: J1.8 (Pin_8), R25.1
- new net OUT4: D5.2 (A), J2.4 (Pin_4), U7.4
- new net OUT5: D6.2 (A), J2.5 (Pin_5), U8.4
- new net OUT8: D9.2 (A), J2.8 (Pin_8), U11.4
- no-connect marks 4 -> 8
Other:
- added sheet 24V-5V again (24V-5V agian.kicad_sch)
- note added: "24+ 24- 24+ 24-"
- note added: "5V CIRCUIT"
- note added: "Arduino"
- note added: "I1 I2 I3 ... I8"
- note added: "IRC5"
- note added: "ISOLATION CIRCUIT"
- note added: "LED"
- note added: "OUTPUT ETHERNET JACK"
- note added: "Overview Schematic"
- note added: "The Plan"
- note added: "This circuit will plug into the din rail of the io modules on the IRC5s in the lab. I plan on having two input plugs and one output plug. The input plugs will include 1 24V input that has anohter plug in parallel to daisy chain voltage out to other modules. Anohter input plug that takes the io signals (at 24V). Those signals will go through an isolator and turn on the other side of the circuit wi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"
- note removed: "Arduino Side"
- note removed: "Rob5000 Side"
- moved on the sheet: D2, Q1, R1, R3, R4, U1
